Commit message: Update Wheel offset

File: firstbot_description/urdf/camera.xacro (robot description, xacro)
@@ -4,5 +4,5 @@
         <parent link="chassis"/>
         <child link="camera_link"/>
-        <origin xyz="0.3 0 0.08" rpy="0 0.18 0"/>
+        <origin xyz="0.3 0 0.05" rpy="0 0.18 0"/>
     </joint>
     <link name="camera_link">

File: firstbot_description/urdf/lidar.xacro (robot description, xacro)
@@ -4,5 +4,5 @@
         <parent link="chassis"/>
         <child link="laser_frame"/>
-        <origin xyz="0.15 0 0.15" rpy="0 0 0"/>
+        <origin xyz="0.15 0 0.10" rpy="0 0 0"/>
     </joint>
     <link name="laser_frame">

File: firstbot_description/urdf/robot_core.xacro (robot description, xacro)
@@ -3,5 +3,5 @@
     <xacro:include filename="inertial_macros.xacro"/>
     <xacro:property name="chassis_length" value="0.3"/>
-    <xacro:property name="chassis_height" value="0.08"/>
+    <xacro:property name="chassis_height" value="0.05"/>
     <xacro:property name="chassis_mass" value="0.5"/>
     <xacro:property name="wheel_radius" value="0.035"/>
@@ -9,6 +9,6 @@
     <xacro:property name="wheel_mass" value="0.05"/>
     <xacro:property name="wheel_offset_x" value="0.15"/>
-    <xacro:property name="wheel_offset_y" value="0.1485"/>
-    <xacro:property name="wheel_offset_z" value="0.01"/>
+    <xacro:property name="wheel_offset_y" value="0.13"/>
+    <xacro:property name="wheel_offset_z" value="-0.02"/>
     <xacro:property name="caster_wheel_radius" value="0.01"/>
     <xacro:property name="caster_wheel_mass" value="0.01"/>
