Commit message: Change lidar height

File: firstbot_description/urdf/lidar.xacro (robot description, xacro)
@@ -4,5 +4,5 @@
         <parent link="chassis"/>
         <child link="laser_frame"/>
-        <origin xyz="0.15 0 0.10" rpy="0 0 0"/>
+        <origin xyz="0.15 0 0.13" rpy="0 0 0"/>
     </joint>
     <link name="laser_frame">
